File: ESP_32_Programer.kicad_pcb (KiCad board)
At the start: 2 copper layers, 37.5 x 13 mm, 21 parts, among them J1 TYPE-C 16PIN 2MD(073), J2 Conn_01x06, Q1 SS8050, Q2 SS8050, U1 CP2102N-A02-GQFN28R, U2 AP2112K-3.3

Commit message: completando PCB
Parts:
- added G***: LOGO, LOGO, F.Cu at (126.5, 96.7)
- added G***: LOGO, LOGO, B.Cu at (126.9, 97.7)
- added R10: 5.1k, Resistor_SMD:R_0603_1608Metric, F.Cu at (131.8, 92.5)
- added R11: 5.1k, Resistor_SMD:R_0603_1608Metric, F.Cu at (131.8, 101.3)
- J1: value TYPE-C 16PIN 2MD(073) -> USB_C_Receptacle_USB2.0_14P
- J2: value Conn_01x06 -> PH2.54-07-03PWS
- Q1, Q2: value SS8050 -> MMBT3904
- R8, R9: footprint Resistor_SMD:R_0603_1608Metric_Pad0.98x0.95mm_HandSolder -> Resistor_SMD:R_0603_1608Metric
- moved R3 1.07 mm to (133.6, 99.3), turned to -45 degrees
- moved R1 0.87 mm to (134.3, 94.2)
- moved R2 0.85 mm to (134.3, 92.7)
- moved R4 0.29 mm to (135.8, 99.3)
- moved R5 0.26 mm to (136.8, 98.2)
Connections:
- J1 pad A5: unconnected-(J1-CC-PadA5) -> Net-(J1-CC1)
- J1 pad A6: Net-(J1-D+) -> Net-(J1-D+-PadA6)
- J1 pad A7: Net-(J1-D-) -> Net-(J1-D--PadA7)
- J1 pad B5: unconnected-(J1-VCONN-PadB5) -> Net-(J1-CC2)
- J1 pad B6: (no net) -> Net-(J1-D+-PadA6)
- J1 pad B7: (no net) -> Net-(J1-D--PadA7)
- R1 pad 1: Net-(J1-D-) -> Net-(J1-D--PadA7)
- R2 pad 1: Net-(J1-D+) -> Net-(J1-D+-PadA6)
Routing:
- net Net-(J1-D+-PadA6): track 0.00 -> 8.56 mm
- net Net-(J1-D--PadA7): track 0.00 -> 7.86 mm, vias 0 -> 2
- net Net-(J1-D+): track 5.91 -> 0.00 mm
- net Net-(J1-D-): track 4.96 -> 0.00 mm
- net Net-(J1-CC2): track 0.00 -> 3.92 mm, vias 0 -> 2
- net Net-(J1-CC1): track 0.00 -> 3.66 mm
- net GND: track 21.2 -> 24.8 mm, vias 15 -> 17
- net VBUS: track 23.2 -> 25.0 mm
- net Net-(U1-D-): track 4.54 -> 3.64 mm
- net Net-(U1-D+): track 4.86 -> 3.98 mm
Other:
- board text added: "${REVISION}"
- board text added: "ESP32"
- board text added: "Prog"
