File: ESP_32_Programer.kicad_pcb (KiCad board)
At the start: 2 copper layers, 37.5 x 13 mm, 25 parts, among them J1 USB_C_Receptacle_USB2.0_14P, J2 PH2.54-07-03PWS, Q1 MMBT3904, Q2 MMBT3904, U1 CP2102N-A02-GQFN28R, U2 AP2112K-3.3

Commit message: actualizando documentacion generando version v1.1.0
Parts:
- removed the G*** at (126.9, 97.7)
Other:
- board text added: "0"
- board text added: "0 mm"
- board text added: "0.0000 mm / 0.0000 mm"
- board text added: "0.01 mm"
- board text added: "0.02"
- board text added: "0.035 mm"
- board text added: "0.3000 mm"
- board text added: "0.91 mm"
- board text added: "1"
- board text added: "1.0000 mm"
- board text added: "2"
- board text added: "3.3"
- board text added: "37.5000 mm x 13.0000 mm"
- board text added: "4.5"
- board text added: "B.Cu"
- board text added: "B.Mask"
- board text added: "B.Paste"
- board text added: "B.Silkscreen"
- board text added: "BOARD CHARACTERISTICS"
- board text added: "Board Thickness:"
- board text added: "Board overall dimensions:"
- board text added: "Bottom Silk Screen"
- board text added: "Bottom Solder Mask"
- board text added: "Bottom Solder Paste"
- board text added: "Castellated pads:"
- board text added: "Color"
- board text added: "Copper Finish:"
- board text added: "Copper Layer Count:"
- board text added: "Dielectric 1"
- board text added: "Direct Printing"
- board text added: "Edge card connectors:"
- board text added: "Epsilon R"
- board text added: "F.Cu"
- board text added: "F.Mask"
- board text added: "F.Paste"
- board text added: "F.Silkscreen"
- board text added: "FR4"
- board text added: "FR4 natural"
- board text added: "Green"
- board text added: "HAL lead-free"
- board text added: "Impedance Control:"
- board text added: "Layer Name"
- board text added: "Liquid Ink"
- board text added: "Lite"
- board text added: "Loss Tangent"
- board text added: "Material"
- board text added: "Min hole diameter:"
- board text added: "Min track/spacing:"
- board text added: "No"
- board text added: "Plated Board Edge:"
- board text added: "Thickness (mm)"
- board text added: "Top Silk Screen"
- board text added: "Top Solder Mask"
- board text added: "Top Solder Paste"
- board text added: "Type"
- board text added: "White"
- board text added: "copper"
- board text added: "core"
